Commit message: fix: align D-task field placement and Gazebo camera

File: src/car_control/urdf/car_sim.urdf.xacro (robot description, xacro)
@@ -85,4 +85,11 @@
     <origin xyz="0 0 0"/>
   </joint>
+  <!-- Physical front-center placement reference: chassis_length_m / 2 ahead of base_link. -->
+  <link name="car_front_reference"/>
+  <joint name="car_front_reference_joint" type="fixed">
+    <parent link="base_link"/>
+    <child link="car_front_reference"/>
+    <origin xyz="${chassis_length_m / 2.0} 0 0" rpy="0 0 0"/>
+  </joint>
   <xacro:wheel side="left" y="${wheel_separation_m / 2.0}"/>
   <xacro:wheel side="right" y="${-wheel_separation_m / 2.0}"/>
